File: TrackMyBike-pcba/power.sch (KiCad schematic (older format))
At the start: 0 parts

Commit message: Add power schematic
Parts:
- added BT?: Battery_Cell, symbol Device:Battery_Cell
- added C? (x2): 47uF, symbol Device:C
- added C?: 1uF, symbol Device:C
- added C? (x2): 1nF, symbol Device:C
- added C?: 10uF, symbol Device:C
- added C?: 100nF, symbol Device:C
- added C?: 10nF, symbol Device:C
- added D?: DIODE, symbol pspice:DIODE
- added D?: SMM4F5.0A-TR, symbol Device:D_Zener
- added J?: Conn_01x02, symbol Connector_Generic:Conn_01x02
- added JP?: 4.2/4.1V, symbol Jumper:SolderJumper_2_Bridged
- added L?: 10uH, symbol Device:L
- added Q?: DMP2165UW, symbol Device:Q_PMOS_GSD
- added Q?: DMN2004WKQ, Package_TO_SOT_SMD:SOT-323_SC-70, symbol Device:Q_NMOS_GSD
- added R? (x2): 10M, symbol Device:R
- added R?: 4.7M, symbol Device:R
- added R? (x3): 1K, symbol Device:R
- added R?: 2.2M, symbol Device:R
- added R?: 820K, symbol Device:R
- added R?: 0R, symbol Device:R
- added R? (x3): DNM, symbol Device:R
- added R? (x2): 100K, symbol Device:R
- added R?: 3.3K, symbol Device:R
- added TH?: Thermistor_NTC, symbol Device:Thermistor_NTC
- added U?: SPV1040T, SOP65P640X120-8N, symbol SPV1040T:SPV1040T
- added U?: L6924D, QFN50P300X300X100-17N, symbol L6924D:L6924D
Connections:
- new net: C?.1, R?.1, R?.2, U?.1 (MPPT-SET)
- new net: L?.2, U?.3 (LX)
- new net: C?.1, C?.1, D?.2 (A), Q?.2 (S), U?.1 (VIN), U?.2 (VINSNS)
- new net: BT?.1 (+), U?.10 (VOSNS), U?.11 (VOUT)
- new net: R?.2, U?.13 (IEND)
- new net: C?.1, U?.5 (TPRG)
- new net: R?.1, TH?.1, U?.8 (TH)
- new net: JP?.1 (A), U?.9 (VOPRG)
- new net +1V0: C?.1, J?.1 (Pin_1), L?.1, R?.2, R?.2
- new net GND: BT?.2 (-), C?.2, C?.2, C?.2, C?.2, C?.2, C?.2, C?.2, D?.2 (A), J?.2 (Pin_2), JP?.2 (B), Q?.2 (S), R?.1, R?.1, R?.1, R?.1, R?.1, R?.1, TH?.2, U?.17 (EP), U?.2 (GND), U?.6 (GND), U?.7 (SD)
- new net ICTRL_MIN: C?.2, R?.1, U?.6 (ICTRL_MINUS)
- new net ICTRL_PLUS: C?.1, R?.1, U?.7 (ICTRL_PLUS)
- new net IPRE: R?.1, R?.2, U?.16 (IPRE)
- new net ST1: U?.4 (ST1)
- new net ST2: U?.3 (ST2)
- new net USB_DET: R?.1, R?.2
- new net VBUS: D?.1 (K), Q?.1 (G), Q?.1 (G), R?.2, R?.2
- new net VCTRL: C?.1, R?.1, R?.2, U?.5 (VCTRL)
- new net VREF: R?.2, R?.2, U?.12 (VREF)
- new net VRS+: D?.1 (K), R?.1, R?.2, U?.4 (VOUT)
- new net VRS-: C?.1, Q?.3 (D), R?.2, R?.2, R?.2
- new net XSHUT: Q?.3 (D), R?.1, U?.8 (XSHUT)
Other:
- note added: "Change pre-charge current\nif required. Default (DNM) \nis 10% of fast-charge current"
- note added: "Connecting VBUS will shut off solar regulator.\nBy default, VBUS is disconnected so that the \ngate is pulled down and the MOSFET is OFF. \nIn this case XSHUT should be pulled up by VSOLAR (if present) \nso that SPV1040 is turned on."
- note added: "MSS7341-103ML"
- note added: "R must be 50mV \n@ Iout(max)\n"
- note added: "USB_DET @3.3V"
- note added: "VOUT=4.2V if VOPRG=GND"
