File: TrackMyBike-pcba/power.sch (KiCad schematic (older format))
At the start: 59 parts

Commit message: Add more footprints
Parts:
- D?: value D -> BAT20JFILM; footprint (none) -> Diode_SMD:D_SOD-323_HandSoldering
Other:
- moved on the sheet: BT?
Changed lines of the file:
@@
 L Device:Battery_Cell BT?
 U 1 1 5F3ABC51
-P 10550 4250
-F 0 "BT?" H 10668 4346 50  0000 L CNN
-F 1 "Battery_Cell" H 10668 4255 50  0000 L CNN
-F 2 "Connector_JST:JST_PH_S2B-PH-SM4-TB_1x02-1MP_P2.00mm_Horizontal" V 10550 4310 50  0001 C CNN
-F 3 "~" V 10550 4310 50  0001 C CNN
-	1    10550 4250
+P 10550 4500
+F 0 "BT?" H 10668 4596 50  0000 L CNN
+F 1 "Battery_Cell" H 10668 4505 50  0000 L CNN
+F 2 "Connector_JST:JST_PH_S2B-PH-SM4-TB_1x02-1MP_P2.00mm_Horizontal" V 10550 4560 50  0001 C CNN
+F 3 "~" V 10550 4560 50  0001 C CNN
+	1    10550 4500
 	1    0    0    -1
 $EndComp
 Wire Wire Line
-	10550 4050 10550 3950
+	10550 4300 10550 3950
 Wire Wire Line
-	10550 4350 10550 5050
+	10550 4600 10550 5050
 Wire Wire Line
 	10550 5050 9850 5050
@@
 P 6050 3950
 F 0 "D?" H 6050 3733 50  0000 C CNN
-F 1 "D" H 6050 3824 50  0000 C CNN
-F 2 "" H 6050 3950 50  0001 C CNN
+F 1 "BAT20JFILM" H 6050 3824 50  0000 C CNN
+F 2 "Diode_SMD:D_SOD-323_HandSoldering" H 6050 3950 50  0001 C CNN
 F 3 "~" H 6050 3950 50  0001 C CNN
 	1    6050 3950
