File: TrackMyBike-pcba/TrackMyBike-pcba.sch (KiCad schematic (older format))
At the start: 1 part, among them J1 USB_B_Micro

Commit message: Modify power.sch, add testpoints
Parts:
- added TP? (x5): TestPoint, symbol Connector:TestPoint
Connections:
- wire segments 10 -> 20
Changed lines of the file:
@@
 $EndSheet
 $Sheet
-S 3450 4800 1350 1250
+S 1500 3700 1350 1250
 U 5F16A6AE
 F0 "Power" 50
 F1 "power.sch" 50
-F2 "ST1" O R 4800 5800 50
-F3 "USB_DET" O R 4800 5700 50
-F4 "ST2" O R 4800 5900 50
-F5 "3V3" O R 4800 5000 50
+F2 "ST1" O R 2850 4150 50
+F3 "USB_DET" O R 2850 4050 50
+F4 "ST2" O R 2850 4250 50
+F5 "3V3" O R 2850 4900 50
+F6 "Vgauge" O R 2850 3950 50
+F7 "SD" O R 2850 3850 50
 $EndSheet
 $Sheet
-S 1500 4800 1400 1400
+S 6900 3650 1400 1400
 U 5F18B9BE
 F0 "Sensors and actuators" 50
@@
 	4050 2050 3050 2050
 Wire Wire Line
-	4800 5000 5300 5000
+	2850 4900 3350 4900
 $Comp
 L power:VSYS #PWR?
 U 1 1 5F3FA9BA
-P 5300 5000
-F 0 "#PWR?" H 5300 4850 50  0001 C CNN
-F 1 "VSYS" H 5315 5173 50  0000 C CNN
-F 2 "" H 5300 5000 50  0001 C CNN
-F 3 "" H 5300 5000 50  0001 C CNN
-	1    5300 5000
+P 3350 4900
+F 0 "#PWR?" H 3350 4750 50  0001 C CNN
+F 1 "VSYS" H 3365 5073 50  0000 C CNN
+F 2 "" H 3350 4900 50  0001 C CNN
+F 3 "" H 3350 4900 50  0001 C CNN
+	1    3350 4900
 	1    0    0    -1
 $EndComp
+Wire Wire Line
+	2850 3950 3150 3950
+Wire Wire Line
+	2850 4050 3250 4050
+Wire Wire Line
+	2850 4150 3350 4150
+Wire Wire Line
+	2850 4250 3450 4250
+$Comp
+L Connector:TestPoint TP?
+U 1 1 5F4B1108
+P 3000 3850
+F 0 "TP?" H 2950 4050 50  0000 L CNN
+F 1 "TestPoint" H 3058 3877 50  0001 L CNN
+F 2 "" H 3200 3850 50  0001 C CNN
+F 3 "~" H 3200 3850 50  0001 C CNN
+	1    3000 3850
+	1    0    0    -1
+$EndComp
+Connection ~ 3000 3850
+Wire Wire Line
+	3000 3850 3100 3850
+Wire Wire Line
+	2850 3850 3000 3850
+$Comp
+L Connector:TestPoint TP?
+U 1 1 5F4B1C32
+P 3150 3950
+F 0 "TP?" H 3100 4150 50  0000 L CNN
+F 1 "TestPoint" H 3208 3977 50  0001 L CNN
+F 2 "" H 3350 3950 50  0001 C CNN
+F 3 "~" H 3350 3950 50  0001 C CNN
+	1    3150 3950
+	1    0    0    -1
+$EndComp
+Connection ~ 3150 3950
+Wire Wire Line
+	3150 3950 3200 3950
+$Comp
+L Connector:TestPoint TP?
+U 1 1 5F4B1F8B
+P 3250 4050
+F 0 "TP?" H 3200 4250 50  0000 L CNN
+F 1 "TestPoint" H 3308 4077 50  0001 L CNN
+F 2 "" H 3450 4050 50  0001 C CNN
+F 3 "~" H 3450 4050 50  0001 C CNN
+	1    3250 4050
+	1    0    0    -1
+$EndComp
+Connection ~ 3250 4050
+Wire Wire Line
+	3250 4050 3300 4050
+$Comp
+L Connector:TestPoint TP?
+U 1 1 5F4B20ED
+P 3350 4150
+F 0 "TP?" H 3300 4350 50  0000 L CNN
+F 1 "TestPoint" H 3408 4177 50  0001 L CNN
+F 2 "" H 3550 4150 50  0001 C CNN
+F 3 "~" H 3550 4150 50  0001 C CNN
+	1    3350 4150
+	1    0    0    -1
+$EndComp
+Connection ~ 3350 4150
+Wire Wire Line
+	3350 4150 3400 4150
+$Comp
+L Connector:TestPoint TP?
+U 1 1 5F4B228D
+P 3450 4250
+F 0 "TP?" H 3400 4450 50  0000 L CNN
+F 1 "TestPoint" H 3508 4277 50  0001 L CNN
+F 2 "" H 3650 4250 50  0001 C CNN
+F 3 "~" H 3650 4250 50  0001 C CNN
+	1    3450 4250
+	1    0    0    -1
+$EndComp
+Connection ~ 3450 4250
+Wire Wire Line
+	3450 4250 3500 4250
 $EndSCHEMATC
